Commit message: Boostrap BB URDF

File: urdf/bb_head.urdf (robot description, URDF)
Before this commit: robot bb_head, 1 links, 0 joints
Links:
- added link camera_link; visual box size=0.01 0.01 0.001
- added link depth_link; visual sphere radius=0.001
- added link front_depth_link; visual box size=0.01 0.01 0.001
- added link left_depth_link; visual box size=0.01 0.01 0.001
- added link right_depth_link; visual box size=0.01 0.01 0.001
- link base_link: geometry visual mesh filename=package://bb_description/meshes/skinny_dome.stl scale=0.0001 0.0001 0.0001
Joints:
- added joint dome_to_camera_joint: type fixed, parent base_link, child camera_link, origin xyz=0 0.12 0.08 rpy=2.093 0 0
- added joint dome_to_depth_joint: type fixed, parent base_link, child depth_link, origin xyz=0 0 0 rpy=0 0 0
- added joint dome_to_front_depth_joint: type fixed, parent base_link, child front_depth_link, origin xyz=0 0.11 0.09 rpy=2.093 0 0
- added joint dome_to_left_depth_joint: type fixed, parent base_link, child left_depth_link, origin xyz=0.11693 -0.067 0.05 rpy=1.047198 0.959931 0.436332
- added joint dome_to_right_depth_joint: type fixed, parent base_link, child right_depth_link, origin xyz=-0.11693 -0.067 0.05 rpy=1.047198 -0.959931 -0.436332

Commit message: Fix dome

File: urdf/bb_head.urdf (robot description, URDF)
Before this commit: robot bb_head, 6 links, 5 joints
Links:
- link base_link: geometry visual mesh filename=package://bb_description/meshes/dome.stl scale=0.0001 0.0001 0.0001

Commit message: Fix up head

File: urdf/bb_head.urdf (robot description, URDF)
Before this commit: robot bb_head, 6 links, 5 joints
Links:
- link base_link: geometry visual mesh filename=package://bb_description/meshes/dome.stl scale=0.001 0.001 0.001
Joints:
- joint dome_to_front_depth_joint: origin xyz=0 0.11 0.09 rpy=2.093 0 0 -> xyz=0 0.11 0.09 rpy=-1.047198 0 0
- joint dome_to_left_depth_joint: origin xyz=0.11693 -0.067 0.05 rpy=1.047198 0.959931 0.436332 -> xyz=0.11693 -0.067 0.05 rpy=1.57075 0.785375 0
- joint dome_to_right_depth_joint: origin xyz=-0.11693 -0.067 0.05 rpy=1.047198 -0.959931 -0.436332 -> xyz=-0.11693 -0.067 0.05 rpy=-1.57075 0.785375 0

Commit message: Fix orientation of sensors

File: urdf/bb_head.urdf (robot description, URDF)
Before this commit: robot bb_head, 6 links, 5 joints
Joints:
- joint dome_to_camera_joint: origin xyz=0 0.12 0.08 rpy=2.093 0 0 -> xyz=0 0.12 0.08 rpy=-1.047198 -0.125826 -3.047137
- joint dome_to_front_depth_joint: origin xyz=0 0.11 0.09 rpy=-1.047198 0 0 -> xyz=0 0.11 0.09 rpy=-1.047198 0 3.14159
- joint dome_to_left_depth_joint: origin xyz=0.11693 -0.067 0.05 rpy=1.57075 0.785375 0 -> xyz=0.122 -0.0715 0.008 rpy=0.5638 1.4933 1.563023
- joint dome_to_right_depth_joint: origin xyz=-0.11693 -0.067 0.05 rpy=-1.57075 0.785375 0 -> xyz=-0.122 -0.0715 0.008 rpy=0.5638 -1.4933 -1.563023

Commit message: Update for rviz rendering

File: urdf/bb_head.urdf (robot description, URDF)
Before this commit: robot bb_head, 6 links, 5 joints
Links:
- added link dome_link; visual mesh filename=package://bb_description/meshes/dome.stl scale=0.001 0.001 0.001
- added link sensor_dish_visual_link; visual mesh filename=package://bb_description/meshes/Radar.stl scale=0.0009 0.0009 0.0009
- added link sensor_link
- link base_link: geometry 
Joints:
- removed joint dome_to_camera_joint
- added joint base_to_dome_joint: type fixed, parent base_link, child dome_link, origin xyz=0 0 0 rpy=0 0 3.14159
- added joint base_to_sensor_joint: type fixed, parent base_link, child sensor_link, origin xyz=.00262 0.1104 0.0709 rpy=-1.028 0 0
- added joint radar_to_camera_joint: type fixed, parent sensor_link, child camera_link, origin xyz=0 0 .002 rpy=0 0 0
- added joint sensor_to_dish_visual_joint: type fixed, parent sensor_link, child sensor_dish_visual_link
- joint dome_to_front_depth_joint: origin xyz=0 0.11 0.09 rpy=-1.047198 0 3.14159 -> xyz=0 -0.015 0.002 rpy=0 0 0; parent base_link -> sensor_link
- joint dome_to_left_depth_joint: origin xyz=0.122 -0.0715 0.008 rpy=0.5638 1.4933 1.563023 -> xyz=0.122 -0.0715 0.008 rpy=0.5638 1.616 0
- joint dome_to_right_depth_joint: origin xyz=-0.122 -0.0715 0.008 rpy=0.5638 -1.4933 -1.563023 -> xyz=-0.122 -0.0715 0.008 rpy=0.5638 -1.616 0
